Commit message: dronecan_node complete and localization

File: urdf/rov.urdf (robot description, URDF)
Before this commit: robot rov, 1 links, 0 joints
Links:
- removed link auv_link
- added link base_link, mass 1.0; collision mesh filename=package://hit25_auv/meshes/rov_urdf.stl scale=0.001 0.001 0.001; visual mesh filename=package://hit25_auv/meshes/rov_urdf.stl scale=0.001 0.001 0.001
