Commit message: khm

File: urdf/rov_rviz_local.urdf (robot description, URDF)
Before this commit: robot rov, 1 links, 0 joints
Links:
- removed link auv_link
- added link base_link, mass 1.0; collision mesh filename=file:///Users/kanghyunmin/Desktop/uuv_sim/rospkg/kmu26_auv/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 scale=0.001 0.001 0.001; visual mesh filename=file:///Users/kanghyunmin/Desktop/uuv_sim/rospkg/kmu26_auv/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 scale=0.001 0.001 0.001
